File: hardware/V5_1_kicad/kinesisBLE V5.kicad_pcb (KiCad board)
At the start: 2 copper layers, 107 x 86 mm, 30 parts, among them J2 CF01131V000, J5_ribbon1 PinHeader_1x10_P2.54mm, J6_ribbon1 PinHeader_1x10_P2.54mm, J7 CF01131V000, X1 JST-XH-02-PIN-ROUND-PAD, X2 JST-XH-02-PIN-ROUND-PAD

Commit message: corrected physical layout
Parts:
- moved X2 80.7 mm to (180.2, 73.4)
- moved R4 47.6 mm to (146.0, 71.0)
- moved R5 45.7 mm to (139.4, 70.9)
- moved X1 12.0 mm to (103.2, 92.9)
- moved U$1 5.00 mm to (122.0, 88.7)
- moved J2 2.00 mm to (194.1, 122.1)
- moved J7 2.00 mm to (103.0, 122.2)
- moved align1 0.50 mm to (108.6, 109.7)
- moved align2 0.50 mm to (188.4, 109.7)
Other:
- board text added: "03.05.21 ver. 5.2"
- board text added: "BUTTON LED"
- board text removed: "14.04.20 ver. 5.1"
- board text removed: "POWER BUTTON"
